File: Beyond_CMoy/Amplifier.kicad_sch (KiCad schematic)
At the start: 51 parts, among them P1 10k, U1 NE5532, U2 NE5532, U3 NE5532, U4 NE5532

Commit message: Layout Board1
Connections:
- net at C9.1, R5.2, R7.1: now also U2.5 (+); no longer U2.3 (+)
- net at C24.2, C27.2, R27.2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: now also U4.2 (-); no longer U4.6 (-)
- net at C13.1, R11.2: now also U2.3 (+); no longer U2.5 (+)
- net at C15.2, C18.2, R17.2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: now also U2.2 (-); no longer U2.6 (-)
- net at C14.1, C15.1, R15.1: now also U2.1; no longer U2.7
- net at C22.1, R21.2: now also U4.3 (+); no longer U4.5 (+)
- net at C23.1, C24.1, R25.1: now also U4.1; no longer U4.7
- net at C10.1, R6.2, R8.1: now also U4.5 (+); no longer U4.3 (+)
- net BIAS_L renamed L_BIAS
- net L_BIAS: now also U2.6 (-), U2.7; no longer U2.1, U2.2 (-)
- net BIAS_R renamed R_BIAS
- net R_BIAS: now also U4.6 (-), U4.7; no longer U4.1, U4.2 (-)
Changed lines of the file:
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@@
 	(wire
 		(pts
-			(xy 255.27 182.88) (xy 255.27 187.96)
+			(xy 255.27 181.61) (xy 255.27 187.96)
 		)
 		(stroke
@@
 		)
 	)
-	(global_label "BIAS_L"
+	(global_label "R_BIAS"
 		(shape output)
-		(at 254 104.14 90)
+		(at 130.81 171.45 90)
 		(fields_autoplaced yes)
 		(effects
@@
 		)
 		(property "Intersheetrefs" "${INTERSHEET_REFS}"
-			(at 254 95.3559 90)
+			(at 130.81 162.5666 90)
 			(effects
 				(font
@@
 		)
 	)
-	(global_label "BIAS_R"
+	(global_label "L_BIAS"
 		(shape output)
-		(at 255.27 182.88 90)
+		(at 80.01 86.36 90)
 		(fields_autoplaced yes)
 		(effects
@@
 		)
 		(property "Intersheetrefs" "${INTERSHEET_REFS}"
-			(at 255.27 173.9966 90)
+			(at 80.01 77.5759 90)
 			(effects
 				(font
@@
 		)
 	)
-	(global_label "BIAS_R"
+	(global_label "L_BIAS"
 		(shape output)
-		(at 130.81 171.45 90)
+		(at 254 104.14 90)
 		(fields_autoplaced yes)
 		(effects
@@
 		)
 		(property "Intersheetrefs" "${INTERSHEET_REFS}"
-			(at 130.81 162.5666 90)
+			(at 254 95.3559 90)
 			(effects
 				(font
@@
 		)
 	)
-	(global_label "BIAS_R"
+	(global_label "R_BIAS"
 		(shape output)
 		(at 80.01 168.91 90)
@@
 		)
 	)
-	(global_label "BIAS_R"
+	(global_label "R_BIAS"
 		(shape output)
-		(at 346.71 57.15 0)
+		(at 255.27 181.61 90)
 		(fields_autoplaced yes)
 		(effects
@@
 		)
 		(property "Intersheetrefs" "${INTERSHEET_REFS}"
-			(at 355.5934 57.15 0)
+			(at 255.27 172.7266 90)
 			(effects
 				(font
@@
 		)
 	)
-	(global_label "BIAS_L"
+	(global_label "R_BIAS"
 		(shape output)
-		(at 130.81 90.17 90)
+		(at 346.71 57.15 0)
 		(fields_autoplaced yes)
 		(effects
@@
 		)
 		(property "Intersheetrefs" "${INTERSHEET_REFS}"
-			(at 130.81 81.3859 90)
+			(at 355.5934 57.15 0)
 			(effects
 				(font
@@
 		)
 	)
-	(global_label "BIAS_L"
+	(global_label "L_BIAS"
 		(shape output)
-		(at 80.01 86.36 90)
+		(at 130.81 90.17 90)
 		(fields_autoplaced yes)
 		(effects
@@
 		)
 		(property "Intersheetrefs" "${INTERSHEET_REFS}"
-			(at 80.01 77.5759 90)
+			(at 130.81 81.3859 90)
 			(effects
 				(font
@@
 		)
 	)
-	(global_label "BIAS_L"
+	(global_label "L_BIAS"
 		(shape output)
 		(at 283.21 57.15 0)
@@
 		(lib_id "Amplifier_Operational:NE5532")
 		(at 270.51 57.15 0)
-		(unit 1)
+		(unit 2)
 		(exclude_from_sim no)
 		(in_bom yes)
@@
 				(path "/1ee317a7-d9f9-4115-84b1-2928dd345c54/2d9672f4-3b4a-4b4e-8c07-73e5cea2fbd1"
 					(reference "U2")
-					(unit 1)
+					(unit 2)
 				)
 			)
@@
 		(lib_id "Amplifier_Operational:NE5532")
 		(at 271.78 123.19 0)
-		(unit 2)
+		(unit 1)
 		(exclude_from_sim no)
 		(in_bom yes)
@@
 				(path "/1ee317a7-d9f9-4115-84b1-2928dd345c54/2d9672f4-3b4a-4b4e-8c07-73e5cea2fbd1"
 					(reference "U2")
-					(unit 2)
+					(unit 1)
 				)
 			)
@@
 		(lib_id "Amplifier_Operational:NE5532")
 		(at 271.78 201.93 0)
-		(unit 2)
+		(unit 1)
 		(exclude_from_sim no)
 		(in_bom yes)
@@
 				(path "/1ee317a7-d9f9-4115-84b1-2928dd345c54/2d9672f4-3b4a-4b4e-8c07-73e5cea2fbd1"
 					(reference "U4")
-					(unit 2)
+					(unit 1)
 				)
 			)
@@
 		(lib_id "Amplifier_Operational:NE5532")
 		(at 335.28 57.15 0)
-		(unit 1)
+		(unit 2)
 		(exclude_from_sim no)
 		(in_bom yes)
@@
 				(path "/1ee317a7-d9f9-4115-84b1-2928dd345c54/2d9672f4-3b4a-4b4e-8c07-73e5cea2fbd1"
 					(reference "U4")
-					(unit 1)
+					(unit 2)
 				)
 			)
