File: Beyond_CMoy/Amplifier.kicad_sch (KiCad schematic)
At the start: 51 parts, among them P1 10k, U1 NE5532, U2 NE5532, U3 NE5532, U4 NE5532

Commit message: PCB Layout
Connections:
- net U1_FB: now reaches C24.2, C27.2, R27.2, R28.2, U4.2 (-)
- net U2_FB: now reaches C15.2, C18.2, R17.2, R18.2, U2.2 (-)
Changed lines of the file:
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@@
+		)
+	)
+	(label "U1_FB"
+		(at 261.62 226.06 0)
+		(effects
+			(font
+				(size 1.27 1.27)
+			)
+			(justify left bottom)
 		)
 	)
@@
 		(effects
 			(font
+				(size 1.27 1.27)
+			)
+			(justify left bottom)
+		)
+	)
+	(label "U2_FB"
+		(at 259.08 147.32 0)
+		(effects
+			(font

Commit message: RELEASED
Parts:
- C10, C9: footprint 0_Devices:0_C_0805_PasteCustom -> 0_Devices:0_C_0805_Edited; Manufacturer Samsung -> SAMSUNG
- C18, C27: footprint 0_Devices:0_C_0805_PasteCustom -> 0_Devices:0_C_0805_Edited
- U1, U2, U3, U4: Manufacturer (none) -> -; Mf. Part Number (none) -> NE5532
Changed lines of the file:
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@@
 			)
 		)
-		(property "Manufacturer" ""
+		(property "Manufacturer" "-"
 			(at 270.51 57.15 0)
 			(effects
@@
 			)
 		)
-		(property "Mf. Part Number" ""
+		(property "Mf. Part Number" "NE5532"
 			(at 270.51 57.15 0)
 			(effects
@@
 			)
 		)
-		(property "Manufacturer" ""
+		(property "Manufacturer" "-"
 			(at 271.78 123.19 0)
 			(effects
@@
 			)
 		)
-		(property "Mf. Part Number" ""
+		(property "Mf. Part Number" "NE5532"
 			(at 271.78 123.19 0)
 			(effects
@@
 			)
 		)
-		(property "Footprint" "0_Devices:0_C_0805_PasteCustom"
+		(property "Footprint" "0_Devices:0_C_0805_Edited"
 			(at 274.0152 223.52 0)
 			(effects
@@
 			)
 		)
-		(property "Manufacturer" ""
+		(property "Manufacturer" "-"
 			(at 146.05 191.77 0)
 			(effects
@@
 			)
 		)
-		(property "Mf. Part Number" ""
+		(property "Mf. Part Number" "NE5532"
 			(at 146.05 191.77 0)
 			(effects
@@
 			)
 		)
-		(property "Manufacturer" ""
+		(property "Manufacturer" "-"
 			(at 99.06 191.77 0)
 			(effects
@@
 			)
 		)
-		(property "Mf. Part Number" ""
+		(property "Mf. Part Number" "NE5532"
 			(at 99.06 191.77 0)
 			(effects
@@
 			)
 		)
-		(property "Manufacturer" ""
+		(property "Manufacturer" "-"
 			(at 99.06 109.22 0)
 			(effects
@@
 			)
 		)
-		(property "Mf. Part Number" ""
+		(property "Mf. Part Number" "NE5532"
 			(at 99.06 109.22 0)
 			(effects
@@
 			)
 		)
-		(property "Manufacturer" ""
+		(property "Manufacturer" "-"
 			(at 271.78 201.93 0)
 			(effects
@@
 			)
 		)
-		(property "Mf. Part Number" ""
+		(property "Mf. Part Number" "NE5532"
 			(at 271.78 201.93 0)
 			(effects
@@
 			)
 		)
-		(property "Manufacturer" ""
+		(property "Manufacturer" "-"
 			(at 99.06 109.22 0)
 			(effects
@@
 			)
 		)
-		(property "Mf. Part Number" ""
+		(property "Mf. Part Number" "NE5532"
 			(at 99.06 109.22 0)
 			(effects
@@
 			)
 		)
-		(property "Footprint" "0_Devices:0_C_0805_PasteCustom"
+		(property "Footprint" "0_Devices:0_C_0805_Edited"
 			(at 244.8052 67.31 0)
 			(effects
@@
 			)
 		)
-		(property "Manufacturer" "Samsung"
+		(property "Manufacturer" "SAMSUNG"
 			(at 243.84 63.5 0)
 			(effects
@@
 			)
 		)
-		(property "Manufacturer" ""
+		(property "Manufacturer" "-"
 			(at 146.05 110.49 0)
 			(effects
@@
 			)
 		)
-		(property "Mf. Part Number" ""
+		(property "Mf. Part Number" "NE5532"
 			(at 146.05 110.49 0)
 			(effects
@@
 			)
 		)
-		(property "Manufacturer" ""
+		(property "Manufacturer" "-"
 			(at 271.78 123.19 0)
 			(effects
@@
 			)
 		)
-		(property "Mf. Part Number" ""
+		(property "Mf. Part Number" "NE5532"
 			(at 271.78 123.19 0)
 			(effects
@@
 			)
 		)
-		(property "Manufacturer" ""
+		(property "Manufacturer" "-"
 			(at 271.78 201.93 0)
 			(effects
@@
 			)
 		)
-		(property "Mf. Part Number" ""
+		(property "Mf. Part Number" "NE5532"
 			(at 271.78 201.93 0)
 			(effects
@@
 			)
 		)
-		(property "Manufacturer" ""
+		(property "Manufacturer" "-"
 			(at 99.06 191.77 0)
 			(effects
@@
 			)
 		)
-		(property "Mf. Part Number" ""
+		(property "Mf. Part Number" "NE5532"
 			(at 99.06 191.77 0)
 			(effects
@@
 			)
 		)
-		(property "Manufacturer" ""
+		(property "Manufacturer" "-"
 			(at 335.28 57.15 0)
 			(effects
@@
 			)
 		)
-		(property "Mf. Part Number" ""
+		(property "Mf. Part Number" "NE5532"
 			(at 335.28 57.15 0)
 			(effects
@@
 			)
 		)
-		(property "Footprint" "0_Devices:0_C_0805_PasteCustom"
+		(property "Footprint" "0_Devices:0_C_0805_Edited"
 			(at 272.7452 144.78 0)
 			(effects
@@
 			)
 		)
-		(property "Footprint" "0_Devices:0_C_0805_PasteCustom"
+		(property "Footprint" "0_Devices:0_C_0805_Edited"
 			(at 308.3052 68.58 0)
 			(effects
@@
 			)
 		)
-		(property "Manufacturer" "Samsung"
+		(property "Manufacturer" "SAMSUNG"
 			(at 307.34 64.77 0)
 			(effects

Commit message: Debugging & New Rev.
Other:
- note added: "0.22uF 0603 X7R"
- note added: "1k"
- note added: "5.1k"
Changed lines of the file:
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@@
 	(title_block
 		(title "Amplifier")
-		(rev "1.0")
+		(rev "1.1")
 		(company "Natchpai")
 	)
@@
 		)
 	)
+	(text "1k"
+		(exclude_from_sim no)
+		(at 151.13 125.73 0)
+		(effects
+			(font
+				(size 12.7 12.7)
+				(thickness 0.762)
+				(bold yes)
+				(color 255 0 0 1)
+			)
+		)
+	)
 	(text "Tantalum"
 		(exclude_from_sim no)
@@
 			(font
 				(size 1.27 1.27)
+			)
+		)
+	)
+	(text "1k"
+		(exclude_from_sim no)
+		(at 149.86 207.01 0)
+		(effects
+			(font
+				(size 12.7 12.7)
+				(thickness 0.762)
+				(bold yes)
+				(color 255 0 0 1)
 			)
 		)
@@
 		)
 	)
+	(text "5.1k"
+		(exclude_from_sim no)
+		(at 252.73 153.67 0)
+		(effects
+			(font
+				(size 12.7 12.7)
+				(thickness 0.762)
+				(bold yes)
+				(color 255 0 0 1)
+			)
+		)
+	)
 	(text "Tantalum\n10V"
 		(exclude_from_sim no)
@@
 			(font
 				(size 1.27 1.27)
+			)
+		)
+	)
+	(text "5.1k"
+		(exclude_from_sim no)
+		(at 254 233.68 0)
+		(effects
+			(font
+				(size 12.7 12.7)
+				(thickness 0.762)
+				(bold yes)
+				(color 255 0 0 1)
 			)
 		)
@@
 			)
 		)
+	)
+	(text "0.22uF 0603 X7R"
+		(exclude_from_sim no)
+		(at 344.17 234.95 0)
+		(effects
+			(font
+				(size 12.7 12.7)
+				(thickness 0.762)
+				(bold yes)
+				(color 255 0 0 1)
+			)
+		)

Commit message: Re-layout
Parts:
- removed C17, C26: 1n, Capacitor_SMD:C_0603_1608Metric, symbol Device:C
- removed C18: 0.22u, 0_Devices:0_C_0805_Edited, symbol Device:C
- removed C20: 0.1u, Capacitor_SMD:C_0402_1005Metric, symbol Device:C
- removed R12, R22: 1k, Resistor_SMD:R_0603_1608Metric, symbol Device:R
- removed R13, R23: 2k, Resistor_SMD:R_0603_1608Metric, symbol Device:R
- removed R19, R20: 100k, Resistor_SMD:R_0603_1608Metric, symbol Device:R
- removed U3: NE5532, Package_SO:SOIC-8_3.9x4.9mm_P1.27mm, symbol Amplifier_Operational:NE5532
- added C19: 0.22u, Capacitor_SMD:C_0603_1608Metric, symbol Device:C
- C26: renamed from C27; footprint 0_Devices:0_C_0805_Edited -> Capacitor_SMD:C_0603_1608Metric
- R15: renamed from R18; value 2k -> 5.1k
- R22: renamed from R28; value 2k -> 5.1k
- renumbered C8 to C10, C9 to C11, C10 to C12, C11 to C13, C12 to C14, C13 to C15, C14 to C16, C15 to C17, C16 to C18, C19 to C20, C28 to C27, C7 to C9, R11 to R10, R14 to R11, R15 to R12, R16 to R13, R17 to R14, R10 to R16, R21 to R17, R24 to R18, R25 to R19, R26 to R20, R27 to R21, U4 to U3
Connections:
- net L_BIAS: no longer R16.2
- net L_BUFFER: now also U1.6 (-)
- net L_IN: now also U1.5 (+); no longer U1.3 (+)
- net R_BIAS: now also R16.2
- net R_BUFFER: now also U1.1, U1.2 (-)
- net R_IN: now also R16.1, U1.3 (+)
- net U2_FB: now also C19.2
- net at R12.2, R14.1: now also C19.1
Other:
- note removed: "0.22uF 0603 X7R"
- note removed: "1k"
- note removed: "5.1k"
- note removed: "U4"
- moved on the sheet: C13, C21, C22, C23, C24, C25, C26, C27, P1A, P1B, R11, R16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
