File: Beyond_CMoy/Beyond_CMoy.kicad_pcb (KiCad board)
At the start: 2 copper layers, 79 x 46 mm, 107 parts, among them J1 PJ-327F, J2 Conn_01x04_Socket, J3 PJ-327F, J4 Conn_01x02_MountingPin, J5 USB_C_Receptacle_PowerOnly_6P, P1 10k, Q1 MMBT3906, U1 NE5532, U2 NE5532, U3 NE5532, U4 NE5532, U5 AP3012, U6 BD50FA1FP3, U7 LP4054HB5F

Commit message: Layout Board1
Parts:
- moved D6 94.1 mm to (112.0, 121.8)
- moved R30 94.1 mm to (115.0, 121.8)
- moved C23 54.4 mm to (151.8, 109.0), turned to 180 degrees
- moved C37 52.1 mm to (172.2, 106.3), turned to -90 degrees
- moved C22 48.9 mm to (157.0, 109.1)
- moved C25 48.0 mm to (147.3, 109.2), turned to 90 degrees
- moved R24 47.7 mm to (127.5, 91.0), turned to 90 degrees
- moved R35 45.9 mm to (175.0, 102.5), turned to 180 degrees
- moved C14 45.7 mm to (132.5, 109.3), turned to 180 degrees
- moved C24 45.6 mm to (152.7, 112.0)
- moved C16 45.4 mm to (128.0, 109.0), turned to 90 degrees
- moved R37 45.1 mm to (176.2, 106.2), turned to -90 degrees
- moved R14 43.9 mm to (129.0, 91.0), turned to 90 degrees
- moved C28 43.1 mm to (153.8, 120.0)
- moved C10 41.8 mm to (163.5, 116.9)
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Connections:
- C10 pad 1: Net-(U4A-+) -> Net-(U4B-+)
- C13 pad 1: Net-(U2B-+) -> Net-(U2A-+)
- C15 pad 2: Net-(U2B--) -> Net-(U2A--)
- C18 pad 2: Net-(U2B--) -> Net-(U2A--)
- C22 pad 1: Net-(U4B-+) -> Net-(U4A-+)
- C24 pad 2: Net-(U4B--) -> Net-(U4A--)
- C27 pad 2: Net-(U4B--) -> Net-(U4A--)
- C9 pad 1: Net-(U2A-+) -> Net-(U2B-+)
- R10 pad 2: BIAS_L -> L_BIAS
- R11 pad 1: BIAS_L -> L_BIAS
- R11 pad 2: Net-(U2B-+) -> Net-(U2A-+)
- R17 pad 2: Net-(U2B--) -> Net-(U2A--)
- R18 pad 2: Net-(U2B--) -> Net-(U2A--)
- R19 pad 2: BIAS_R -> R_BIAS
- R20 pad 2: BIAS_R -> R_BIAS
- R21 pad 1: BIAS_R -> R_BIAS
- R21 pad 2: Net-(U4B-+) -> Net-(U4A-+)
- R27 pad 2: Net-(U4B--) -> Net-(U4A--)
- R28 pad 2: Net-(U4B--) -> Net-(U4A--)
- R5 pad 2: Net-(U2A-+) -> Net-(U2B-+)
- R6 pad 2: Net-(U4A-+) -> Net-(U4B-+)
- R7 pad 1: Net-(U2A-+) -> Net-(U2B-+)
- R8 pad 1: Net-(U4A-+) -> Net-(U4B-+)
- R9 pad 2: BIAS_L -> L_BIAS
- U2 pad 1: BIAS_L -> Net-(C14-Pad1)
- U2 pad 2: BIAS_L -> Net-(U2A--)
- U2 pad 6: Net-(U2B--) -> L_BIAS
- U2 pad 7: Net-(C14-Pad1) -> L_BIAS
- U4 pad 1: BIAS_R -> Net-(C23-Pad1)
- U4 pad 2: BIAS_R -> Net-(U4A--)
- U4 pad 6: Net-(U4B--) -> R_BIAS
- U4 pad 7: Net-(C23-Pad1) -> R_BIAS
Other:
- board text added: "Beyond"
- board text added: "CMoy"

Commit message: PCB Layout
Parts:
- moved C27 40.9 mm to (126.0, 148.0)
- moved R6 40.9 mm to (139.2, 146.5), turned to -90 degrees
- moved R8 40.6 mm to (137.8, 146.5), turned to -90 degrees
- moved C8 40.4 mm to (138.8, 144.5), turned to 0 degrees
- moved C10 40.4 mm to (136.0, 146.5), turned to -90 degrees
- moved C23 40.0 mm to (125.0, 138.8)
- moved C25 40.0 mm to (120.5, 139.0)
- moved R26 40.0 mm to (121.8, 138.6)
- moved R27 40.0 mm to (126.0, 144.8)
- moved R25 39.9 mm to (126.0, 143.2), turned to 180 degrees
- moved C24 39.9 mm to (126.0, 141.8), turned to 180 degrees
- moved U4 38.8 mm to (131.2, 143.6)
- moved C22 38.6 mm to (130.5, 137.1), turned to 90 degrees
- moved C21 38.5 mm to (135.5, 141.2), turned to 90 degrees
- moved C28 35.8 mm to (131.8, 148.2)
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Routing:
- net Net-(U4A-+): track 0.00 -> 4.11 mm
- net R_BIAS: track 0.00 -> 3.44 mm
- net +9VA: track 0.00 -> 2.19 mm, vias 0 -> 1

Commit message: PCB Layout
Parts:
- moved C33 13.3 mm to (144.0, 83.5)
- moved C34 13.3 mm to (141.0, 83.5)
- moved U6 13.3 mm to (142.5, 88.2)
- moved TP4 12.6 mm to (146.2, 96.0)
- moved R14 2.75 mm to (129.0, 88.2)
- moved R24 2.75 mm to (127.5, 88.2)
- moved C20 1.23 mm to (130.5, 109.0), turned to 180 degrees
- moved C6 1.00 mm to (115.0, 94.0)
- moved D2 1.00 mm to (114.5, 95.5)
- moved C26 0.90 mm to (133.0, 107.2)
- moved R19 0.90 mm to (136.5, 114.8), turned to -90 degrees
- moved R20 0.90 mm to (136.5, 111.7)
- moved R23 0.90 mm to (133.0, 108.8)
- moved U3 0.90 mm to (133.0, 113.2)
- moved R10 0.76 mm to (136.5, 99.8)
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Routing:
- net /Interface/R_JACK: track 0.00 -> 15.8 mm
- net /Interface/L_JACK: track 0.00 -> 14.0 mm
- net Net-(U3B--): track 0.00 -> 9.85 mm
- net Net-(U1B--): track 0.00 -> 9.85 mm
- net /Interface/R_BT: track 0.00 -> 7.18 mm
- net Net-(U3A--): track 0.00 -> 7.10 mm
- net Net-(U1A--): track 0.00 -> 6.96 mm
- net L_BIAS: track 0.00 -> 5.06 mm
- net R_BIAS: track 3.44 -> 8.38 mm
- net /Interface/L_COUP: track 0.00 -> 4.38 mm
- net Net-(U1B-+): track 0.00 -> 4.38 mm
- net /Interface/R_COUP: track 0.00 -> 4.37 mm
- net Net-(U3B-+): track 0.00 -> 4.23 mm
- net /Interface/L_BT: track 0.00 -> 4.09 mm
- net /Amplifier/R_BUFFER: track 0.00 -> 3.62 mm
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
Commit message: PCB Layout
Parts:
- moved R6 43.3 mm to (144.4, 103.5), turned to 0 degrees
- moved R8 42.0 mm to (144.4, 105.0), turned to 0 degrees
- moved C8 40.7 mm to (142.4, 104.0), turned to 90 degrees
- moved C10 40.6 mm to (144.4, 106.7), turned to 0 degrees
- moved C28 40.0 mm to (146.1, 110.9), turned to 90 degrees
- moved C27 37.0 mm to (145.9, 116.7), turned to 90 degrees
- moved C9 36.4 mm to (162.2, 105.8), turned to 90 degrees
- moved TP1 35.3 mm to (150.5, 75.8)
- moved R7 35.0 mm to (160.5, 105.8), turned to 90 degrees
- moved R28 34.6 mm to (144.1, 116.7), turned to -90 degrees
- moved C21 34.2 mm to (139.1, 107.2), turned to 180 degrees
- moved R5 34.0 mm to (159.0, 105.8), turned to 90 degrees
- moved U4 33.7 mm to (141.5, 111.5), turned to 90 degrees
- moved C7 32.7 mm to (157.6, 106.0), turned to -90 degrees
- moved R27 32.6 mm to (142.6, 116.7), turned to 90 degrees
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Routing:
- net Net-(J5-CC2): track 0.00 -> 15.4 mm
- net Net-(J5-CC1): track 0.00 -> 12.4 mm
- net R_BIAS: track 8.38 -> 0.00 mm
- net Net-(D9-A): track 0.00 -> 7.04 mm
- net /Interface/R_COUP: track 4.37 -> 0.00 mm
- net Net-(D8-A): track 0.00 -> 4.11 mm
- net L_BIAS: track 5.06 -> 1.35 mm
- net +9VA: track 2.19 -> 5.35 mm, vias 1 -> 2
- net /Battery Management System/STAT1: track 0.00 -> 2.51 mm
- net Net-(U4A-+): track 4.11 -> 1.92 mm
- net Net-(U1B--): track 9.85 -> 9.22 mm
- net Net-(U3B--): track 9.85 -> 9.29 mm

Commit message: PCB Layout
Parts:
- moved C16 31.1 mm to (125.8, 110.2), turned to -90 degrees
- moved C25 12.4 mm to (125.8, 116.8), turned to -90 degrees
- moved R11 11.7 mm to (153.4, 107.2)
- moved C19 4.94 mm to (163.6, 112.0)
- moved R26 4.74 mm to (140.0, 117.8), turned to -90 degrees
- moved R18 4.19 mm to (161.9, 117.7), turned to -90 degrees
- moved R6 3.51 mm to (144.5, 107.0), turned to 90 degrees
- moved C10 3.37 mm to (147.8, 107.0), turned to 90 degrees
- moved R16 3.34 mm to (155.9, 117.7), turned to -90 degrees
- moved C8 3.15 mm to (143.2, 107.0), turned to -90 degrees
- moved C22 2.66 mm to (137.5, 111.2), turned to -90 degrees
- moved R8 2.57 mm to (146.0, 107.0), turned to 90 degrees
- moved R21 2.51 mm to (137.5, 107.2)
- moved C27 2.12 mm to (147.8, 117.8)
- moved R28 2.12 mm to (146.0, 117.8)
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Routing:
- net +9VA: track 5.35 -> 14.7 mm, vias 2 -> 6
- net Net-(U4A-+): track 1.92 -> 0.00 mm

Commit message: RELEASED
Parts:
- removed the C35 at (177.0, 97.0)
- added ?: , , F.Cu at (186.0, 82.0)
- added C36: 10u, Capacitor_SMD:C_1206_3216Metric, F.Cu at (177.2, 102.0)
- added C38: 0.1u, Capacitor_SMD:C_0402_1005Metric, F.Cu at (176.3, 111.3)
- added C39: 0.1u, Capacitor_SMD:C_0402_1005Metric, F.Cu at (172.0, 107.9)
- added D10: RED, LED_SMD:LED_0603_1608Metric, F.Cu at (186.7, 121.1)
- added G***: LOGO, LOGO, B.Cu at (186.8, 113.4)
- added G1: LOGO, LOGO, F.Cu at (159.1, 118.1)
- added R41: 2k, Resistor_SMD:R_0603_1608Metric, F.Cu at (183.3, 121.1)
- added R42: 100k, Resistor_SMD:R_0603_1608Metric, F.Cu at (170.1, 112.5)
- added R43: 10k, Resistor_SMD:R_0603_1608Metric, F.Cu at (170.1, 111.0)
- added R44: 62k, Resistor_SMD:R_0603_1608Metric, F.Cu at (170.1, 114.0)
- added TP6: GND, TestPoint:TestPoint_THTPad_1.5x1.5mm_Drill0.7mm, F.Cu at (165.1, 102.0)
- added TP8: GND, TestPoint:TestPoint_THTPad_1.5x1.5mm_Drill0.7mm, F.Cu at (159.5, 89.9)
- added U8: BA8391G-TR, Package_TO_SOT_SMD:SOT-23-5, F.Cu at (173.7, 111.8)
- added U9: TL432ASF, Package_TO_SOT_SMD:SOT-23, F.Cu at (169.5, 108.4)
- C10, C18, C27, C29, C30, C31, C32, C33, C34, C9: footprint 0_Devices:0_C_0805_PasteCustom -> 0_Devices:0_C_0805_Edited
- C37: footprint Capacitor_SMD:C_Elec_5x5.4 -> Capacitor_SMD:C_1206_3216Metric
- D6: footprint LED_SMD:LED_0603_1608Metric -> LED_SMD:LED_Kingbright_APA1606_1.6x0.6mm_Horizontal
- L1: value 4.7uH -> 10u; footprint Inductor_SMD:L_0603_1608Metric -> 0_Devices:0_L_1008_Edited
- R35: value 0 -> 1
- TP5: footprint TestPoint:TestPoint_Pad_D2.0mm -> TestPoint:TestPoint_Pad_D1.0mm
- moved TP1 27.3 mm to (168.7, 96.1), turned to 180 degrees
- moved TP2 24.8 mm to (160.6, 97.2), turned to 0 degrees
- moved C13 23.4 mm to (130.0, 110.5), turned to 90 degrees
- moved C14 23.4 mm to (130.0, 117.3)
- moved C15 23.3 mm to (134.0, 118.2)
- moved R15 23.3 mm to (135.5, 118.2)
- moved R16 23.3 mm to (132.5, 118.2)
- moved R17 23.3 mm to (137.0, 118.2)
- moved R18 23.3 mm to (138.5, 118.2)
- moved C18 23.3 mm to (140.3, 118.2)
- moved U2 22.9 mm to (136.2, 113.0)
- moved C12 22.9 mm to (133.9, 108.8)
- moved C19 22.9 mm to (140.8, 112.5)
- moved C7 22.9 mm to (136.2, 107.7), turned to 90 degrees
- moved C9 22.9 mm to (140.8, 107.7), turned to -90 degrees
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- renumbered C36 to C35
Connections:
- net Net-(U2A--) renamed /Amplifier/U2_FB
- net Net-(U4A--) renamed /Amplifier/U1_FB
- C37 pad 1: Net-(C37-Pad1) -> +BATT
- P1 pad 7: GND -> /Interface/Power_ON
- P1 pad 8: /Interface/Power_ON -> GND
- R35 pad 2: Net-(C37-Pad1) -> Net-(C36-Pad1)
Routing:
- net +9VA: track 14.7 -> 173.0 mm, vias 6 -> 7
- net +BATT: track 0.00 -> 98.4 mm
- net /Interface/R_COUP: track 0.00 -> 64.2 mm
- net /Interface/R_OUT: track 0.00 -> 62.5 mm
- net /Interface/Power_ON: track 0.00 -> 54.6 mm, vias 0 -> 2
- net /Amplifier/R_ATT: track 0.00 -> 47.8 mm, vias 0 -> 2
- net GND: track 0.01 -> 46.7 mm, vias 0 -> 168
- net /Battery Management System/STAT1: track 2.51 -> 45.8 mm, vias 0 -> 2
- net /Amplifier/R_BUFFER: track 3.62 -> 42.2 mm, vias 0 -> 4
- net +9V: track 0.00 -> 34.6 mm
- net /Amplifier/L_ATT: track 0.00 -> 34.2 mm, vias 0 -> 2
- net /Interface/L_COUP: track 4.76 -> 38.4 mm
- net VBUS: track 0.00 -> 33.2 mm
- net R_BIAS: track 0.00 -> 32.9 mm
- net L_BIAS: track 1.35 -> 34.1 mm, vias 0 -> 4
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- added copper zone on F.Cu, net +9V
- added copper zone on F.Cu, net +BATT
- added copper zone on F.Cu, net /Power Management System/BS_SW
- added copper zone on B.Cu, net GND
- added copper zone on F.Cu, net GND
- added copper zone on F.Cu, net VBUS
Other:
- board size 79 x 46 mm -> 79 x 47 mm
- board text added: "(0, 0)"
- board text added: "0.010mm"
- board text added: "0.035mm"
- board text added: "0.150mm"
- board text added: "0.2000 mm / 0.2000 mm"
- board text added: "0.3000 mm"
- board text added: "0.30mm"
- board text added: "0.40mm"
- board text added: "0.50mm"
- board text added: "0.70mm"
- board text added: "1"
- board text added: "1.00mm"
- board text added: "1.50mm"
- board text added: "1.51mm"
- board text added: "1.6000 mm"
- board text added: "12"
- board text added: "12-2025 Rev1.0"
- board text added: "190"
- board text added: "2"
- board text added: "2.00mm"
- board text added: "4"
- board text added: "5"
- board text added: "5V"
- board text added: "79.0000 mm x 47.0000 mm"
- board text added: "9V"
- board text added: "9VA"
- board text added: "AA-2025-11-001-M1"
- board text added: "ASSEMPLY NOTE 1. Don't populate parts are marked with a red cross."
- board text added: "Amplifier & Li-Po Battery Charger"
- board text added: "B.Cu"
- board text added: "B.Silk screen"
- board text added: "B.Solder Mask"
- board text added: "BATT"
- board text added: "BOARD CHARACTERISTICS"
- board text added: "Board Thickness:"
- board text added: "Board overall dimensions:"
- board text added: "Bottom Fabrication (Scale 1:1)"
- board text added: "Bottom Layer (SIG/PWR/GND)"
- board text added: "COPPER"
- board text added: "CORE"
- board text added: "Castellated pads:"
- board text added: "Chr"
- board text added: "Copper Finish:"
- board text added: "Copper Layer Count:"
- board text added: "Count"
- board text added: "DESIGN GEOMETRY MINIMUM FEATURE SIZES: TRACE WIDTH 0.20 mm TRACE TO TRACE 0.20 mm MIN. HOLE (PTH) 0.30 mm MIN. HOLE (NPTH) 0.30 mm MIN. ANNULAR RING 0.15 mm MIN. VIA DIAMETER 0.60 mm COPPER TO HOLE 0.25 mm COPPER TO EDGE 0.50 mm HOLE TO HOLE 0.25 mm"
- board text added: "Drill Map (Scale 1:1)"
- board text added: "Edge card connectors:"
- board text added: "F.Cu"
- board text added: "F.Silk Screen"
- board text added: "F.Solder Mask"
- board text added: "F.Solder Paste"
- board text added: "Full"
- board text added: "GND"
- board text added: "HAL SnPb"
- board text added: "INPUT"
- board text added: "Impedance Control:"
- board text added: "Low"
- board text added: "Material"
- board text added: "Min hole diameter:"
- board text added: "Min track/spacing:"
- board text added: "Name"
- board text added: "No"
- board text added: "Non-Plated"
- board text added: "OUTPUT"
- board text added: "PWR"
- board text added: "Plate"
- board text added: "Plated"
- board text added: "Plated Board Edge:"
- board text added: "RF4 TG135"
- board text added: "Ref. Net X[mm.] Y[mm.]"
- board text added: "Size"
- board text added: "Symbol"
- board text added: "TP1 +BATT 58.70 29.90"
- board text added: "TP2 +9VA 50.60 28.80"
- board text added: "TP3 +9V 49.70 42.7"
- board text added: "TP4 +5V 32.00 38.5"
- board text added: "TP5 USB 70.90 15.80"
- board text added: "TP6 GND 55.10 24.00"
- board text added: "TP7 *** *** ***"
- board text added: "TP8 GND 49.50 36.1"
- board text added: "Thickness"
- board text added: "Top Dimension (Scale 1:1)"
- board text added: "Top Fabrication (Scale 1:1)"
- board text added: "Top Layer (SIG/PWR/GND)"
- board text added: "U1"
- board text added: "U2"
- board text added: "U3"
- board text added: "U4"
- board text added: "U5"
- board text added: "U6"
- board text added: "USB"
- board text added: "X"
- board text added: "Y"
- board text removed: "Drill Origin"
- board text removed: "FABRICATION NOTES (UNLESS OTHERWISE SPECIFIED) 1) OUTLINE DEFINED IN SEPARATE GERBER FILE WITH {dblquote}Edge_Cuts.GBR{dblquote} SUFFIX. DIMENSIONS OF CIRCUMSIZED RECTANGLE SHOWN ON THIS DWG FOR REF ONLY. 2) SEE SEPARATE DRILL FILES WITH {dblquote}.DRL{dblquote} SUFFIX FOR HOLE LOCATIONS. SELECTED HOLE LOCATIONS SHOWN ON THIS DWG FOR REF ONLY. 3) IMPEDANCE CONTROL REQUIRED. Microstrip 100-Ohm Dif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"
- board text removed: "Top Dimention (Scale 1:1)"

Commit message: Debugging & New Rev.
Connections:
- U6 pad 1: +9V -> +5V
- U6 pad 3: +5V -> +9V
Routing:
- net +9V: track 34.6 -> 30.2 mm
- net +5V: track 17.7 -> 13.6 mm
Changed lines of the file:
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@@
 			(layers "F.Cu" "F.Mask" "F.Paste")
 			(roundrect_rratio 0.25)
-			(net 29 "+9V")
-			(pinfunction "VCC")
-			(pintype "power_in")
+			(net 31 "+5V")
+			(pinfunction "VO")
+			(pintype "power_out")
 		)
 		(pad "2" smd custom
@@
 			(layers "F.Cu" "F.Mask" "F.Paste")
 			(roundrect_rratio 0.25)
-			(net 31 "+5V")
-			(pinfunction "VO")
-			(pintype "power_out")
+			(net 29 "+9V")
+			(pinfunction "VCC")
+			(pintype "power_in")
 		)
 		(embedded_fonts no)
@@
 	)
 	(segment
-		(start 148.5 84.85)
-		(end 148.5 86.6125)
-		(width 0.5)
-		(layer "F.Cu")
-		(net 29)
-	)
-	(segment
 		(start 159.75 83.35)
 		(end 161.4 85)
@@
 	)
 	(segment
-		(start 148.5 84.85)
-		(end 151.15 84.85)
-		(width 0.5)
-		(layer "F.Cu")
-		(net 29)
-	)
-	(segment
 		(start 161.75 89.25)
 		(end 162 89.5)
@@
 		(width 0.5)
 		(layer "F.Cu")
-		(net 31)
-	)
-	(segment
-		(start 145.5 84.95)
-		(end 145.5 86.6125)
-		(width 0.5)
-		(layer "F.Cu")
-		(net 31)
-	)
-	(segment
-		(start 143.0125 86.6125)
-		(end 145.5 86.6125)
-		(width 0.5)
-		(layer "F.Cu")
