File: Beyond_CMoy/Beyond_CMoy.kicad_pcb (KiCad board)
At the start: 2 copper layers, 79 x 47 mm, 121 parts, among them J1 PJ-327F, J2 Conn_01x04_Socket, J3 PJ-327F, J4 Conn_01x02_MountingPin, J5 USB_C_Receptacle_PowerOnly_6P, P1 10k, Q1 MMBT3906, U1 NE5532, U2 NE5532, U3 NE5532, U4 NE5532, U5 AP3012, U6 BD50FA1FP3, U7 LP4054HB5F, U8 BA8391G-TR, U9 TL432ASF

Commit message: Re-layout
Parts:
- removed ?: , 
- removed the C17 at (136.4, 94.0)
- removed the C18 at (140.3, 118.2)
- removed the C20 at (150.6, 95.8)
- removed the C26 at (153.2, 94.0)
- removed the R12 at (132.8, 100.0)
- removed the R13 at (136.4, 95.5)
- removed the R19 at (156.5, 101.5)
- removed the R20 at (156.5, 98.4)
- removed the R22 at (149.5, 100.0)
- removed the R23 at (153.2, 95.5)
- removed the R31 at (174.2, 91.8)
- removed the U3 at (153.0, 100.0)
- removed the U6 at (147.0, 88.6)
- added C19: 0.22u, Capacitor_SMD:C_0603_1608Metric, F.Cu at (140.0, 118.2)
- added C2: 33p, Capacitor_SMD:C_0402_1005Metric, F.Cu at (129.5, 85.0)
- added C31: 0.1u, Capacitor_SMD:C_0402_1005Metric, F.Cu at (179.4, 84.0)
- added C4: 33p, Capacitor_SMD:C_0402_1005Metric, F.Cu at (129.5, 83.5)
- added U5: BD50FA1FP3-ZTL, Package_TO_SOT_SMD:SOT-89-3, F.Cu at (146.8, 84.3)
- C26: renamed from C27; footprint 0_Devices:0_C_0805_Edited -> Capacitor_SMD:C_0603_1608Metric
- D7: footprint Diode_SMD:D_SOD-923 -> 0_Devices:D_SOD-923_Edited
- Q1: value MMBT3906 -> AO3401A; footprint Package_TO_SOT_SMD:SOT-23 -> Package_TO_SOT_SMD:SOT-23-3
- R15: renamed from R18; value 2k -> 5.1k
- R22: renamed from R28; value 2k -> 5.1k
- R23: renamed from R29; value 0 -> 1M
- R27: renamed from R34; value 5.1k -> 0
- TP5: renamed from TP4; footprint TestPoint:TestPoint_Pad_D2.0mm -> TestPoint:TestPoint_Pad_D1.0mm
- moved TP1 10.7 mm to (151.7, 91.3)
- moved Q1 8.32 mm to (175.1, 84.0)
- moved R23 7.39 mm to (178.1, 84.0), turned to -90 degrees
- moved C33 5.06 mm to (148.2, 89.0), turned to -90 degrees
- moved C34 4.96 mm to (145.2, 89.0), turned to -90 degrees
- moved R27 3.98 mm to (175.5, 86.5), turned to 180 degrees
- moved R9 3.07 mm to (140.5, 98.6), turned to 0 degrees
- moved R16 2.92 mm to (140.5, 101.4), turned to 0 degrees
- moved R11 2.50 mm to (128.2, 91.5)
- moved R18 2.50 mm to (128.2, 89.5)
- moved C7 2.25 mm to (126.5, 100.6)
- moved R4 2.25 mm to (126.5, 104.4)
- moved C5 2.20 mm to (124.3, 100.6)
- moved R3 2.20 mm to (124.3, 104.4)
- moved C28 1.05 mm to (155.4, 86.8)
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- renumbered C8 to C10, C9 to C11, C10 to C12, C11 to C13, C12 to C14, C13 to C15, C14 to C16, C15 to C17, C16 to C18, C19 to C20, C28 to C27, C30 to C28, C31 to C29, C2 to C3, C29 to C30, C3 to C5, C4 to C6, C5 to C7, C6 to C8, C7 to C9, J2 to J1, J1 to J2, R11 to R10, R14 to R11, R15 to R12, R16 to R13, R17 to R14, R10 to R16, R21 to R17, R24 to R18, R25 to R19, R26 to R20, R27 to R21, R30 to R24, R33 to R25, R32 to R26, R35 to R28, R36 to R29, R37 to R30, R38 to R31, R39 to R32, R40 to R33, R41 to R34, R42 to R35, R43 to R36, R44 to R37, TP2 to TP1, TP1 to TP2, TP6 to TP3, TP3 to TP4, TP8 to TP6, TP5 to TP7, U4 to U3, U5 to U4, U7 to U6, U8 to U7, U9 to U8
Connections:
- C32 pad 1: +BATT -> /Power Management System/ON_BATT
- L1 pad 1: +BATT -> /Power Management System/ON_BATT
- Q1 pad 1: Net-(Q1-B) -> /Power Management System/FET_G
- Q1 pad 3: /Power Management System/BS_EN -> /Power Management System/ON_BATT
- R16 pad 1: Net-(U1B-+) -> /Interface/R_COUP
- R16 pad 2: L_BIAS -> R_BIAS
- R23 pad 1: /Power Management System/BS_EN -> +BATT
- R23 pad 2: +BATT -> /Power Management System/FET_G
- R27 pad 1: Net-(Q1-B) -> /Power Management System/FET_G
- U1 pad 1: Net-(U1A--) -> /Amplifier/R_BUFFER
- U1 pad 2: Net-(U1A--) -> /Amplifier/R_BUFFER
- U1 pad 3: /Interface/L_COUP -> /Interface/R_COUP
- U1 pad 5: Net-(U1B-+) -> /Interface/L_COUP
- U1 pad 6: Net-(U1B--) -> /Amplifier/L_BUFFER
- U4 pad 4: /Power Management System/BS_EN -> /Power Management System/ON_BATT
- U4 pad 5: +BATT -> /Power Management System/ON_BATT
Routing:
- net /Interface/R_COUP: track 64.2 -> 32.0 mm
- net Net-(Q1-B): track 18.0 -> 0.00 mm, vias 2 -> 0
- net /Power Management System/ON_BATT: track 0.00 -> 17.5 mm
- net /Amplifier/R_BUFFER: track 42.2 -> 27.3 mm
- net +BATT: track 98.4 -> 84.1 mm
- net GND: track 46.7 -> 33.2 mm, vias 168 -> 177
- net +9VA: track 173.0 -> 161.7 mm
- net R_BIAS: track 32.9 -> 23.0 mm
- net Net-(U3B--): track 9.29 -> 0.00 mm
- net Net-(U1B--): track 9.22 -> 0.00 mm
- net /Power Management System/BS_EN: track 8.75 -> 0.00 mm
- net /Interface/L_COUP: track 38.4 -> 30.4 mm
- net +5V: track 13.6 -> 21.1 mm, vias 1 -> 0
- net Net-(U3A--): track 7.15 -> 0.00 mm
- net Net-(U1A--): track 6.90 -> 0.00 mm
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- added copper zone on F.Cu, net /Power Management System/ON_BATT
