File: Beyond_CMoy/BMS.kicad_sch (KiCad schematic)
At the start: 16 parts, among them J4 Conn_01x02_MountingPin, J5 USB_C_Receptacle_PowerOnly_6P, U7 LP4054HB5F

Commit message: PCB Layout
Other:
- note added: "C0G"
Changed lines of the file:
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@@
+		)
+	)
+	(text "C0G"
+		(exclude_from_sim no)
+		(at 100.584 84.836 0)
+		(effects
+			(font
+				(size 1.27 1.27)
+			)
 		)
 	)

Commit message: RELEASED
Parts:
- removed C35, C37: 10u, Capacitor_SMD:C_Elec_5x5.4, symbol Device:C_Polarized
- added C36, C37: 10u, Capacitor_SMD:C_1206_3216Metric, symbol Device:C
- added C38, C39: 0.1u, Capacitor_SMD:C_0402_1005Metric, symbol Device:C
- added D10: RED, LED_SMD:LED_0603_1608Metric, symbol Device:LED
- added R41: 2k, Resistor_SMD:R_0603_1608Metric, symbol Device:R
- added R42: 100k, Resistor_SMD:R_0603_1608Metric, symbol Device:R
- added R43: 10k, Resistor_SMD:R_0603_1608Metric, symbol Device:R
- added R44: 62k, Resistor_SMD:R_0603_1608Metric, symbol Device:R
- added U8: BA8391G-TR, Package_TO_SOT_SMD:SOT-23-5, symbol 0_BA8391G-TR:BA8391G-TR
- added U9: TL432ASF, Package_TO_SOT_SMD:SOT-23, symbol Reference_Voltage:TL432DBZ
- J4: Manufacturer - -> JST; Mf. Part Number (none) -> PHCONNECTOR
- R35: value 0 -> 1; Mf. Part Number 0603WAF0000T5E -> 0603WAF100KT5E
- TP5: footprint TestPoint:TestPoint_Pad_D2.0mm -> TestPoint:TestPoint_Pad_D1.0mm
- U7: Manufacturer (none) -> LPS; Mf. Part Number (none) -> LP4054H
- renumbered C36 to C35
Connections:
- net +BATT: now also C37.1, C38.1, R41.1, R42.1, R43.1, U8.5 (V+)
- net GND: now also C36.2, C37.2, C38.2, C39.1, R44.2, U8.2 (V-), U9.3 (A)
- net at R35.2: now also C36.1
- new net: C39.2, R43.2, U8.1 (-), U9.1 (REF), U9.2 (K)
- new net: R42.2, R44.1, U8.3 (+)
- new net: D10.1 (K), U8.4
- new net: D10.2 (A), R41.2
Other:
- note added: "1.24V"
- note added: "Low Battery Monitor"
- note added: "Trigger around +VBATT 3.24V"
- moved on the sheet: C35, D7, D8, D9, J4, J5, R35, R36, R37, R38, R39, R40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

Commit message: Update Doc and Same verison Release
Release v1.0 , Update Doc Files
Parts:
- J4: Mf. Part Number PHCONNECTOR -> S2B-PH-SM4-TB

Commit message: Re-layout
Parts:
- D7: footprint Diode_SMD:D_SOD-923 -> 0_Devices:D_SOD-923_Edited
- renumbered R35 to R28, R36 to R29, R37 to R30, R38 to R31, R39 to R32, R40 to R33, R41 to R34, R42 to R35, R43 to R36, R44 to R37, TP5 to TP7, U7 to U6, U8 to U7, U9 to U8
Other:
- note added: "Low-Battery Monitor"
- note removed: "Low Battery Monitor"
Changed lines of the file:
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@@
 		)
 	)
-	(text "Low Battery Monitor"
+	(text "Low-Battery Monitor"
 		(exclude_from_sim no)
-		(at 259.08 111.76 0)
+		(at 220.98 158.75 0)
 		(effects
 			(font
@@
 		(dnp no)
 		(fields_autoplaced yes)
-		(property "Reference" "#PWR065"
+		(property "Reference" "#PWR062"
 			(at 176.53 120.65 0)
 			(effects
@@
 			(project "Beyond_CMoy"
 				(path "/1ee317a7-d9f9-4115-84b1-2928dd345c54/615c305d-8768-47e7-86f6-9adb9bcb9cb4"
-					(reference "#PWR065")
+					(reference "#PWR062")
 					(unit 1)
 				)
@@
 		(dnp no)
 		(fields_autoplaced yes)
-		(property "Reference" "#PWR066"
+		(property "Reference" "#PWR061"
 			(at 213.36 118.11 0)
 			(effects
@@
 			(project "Beyond_CMoy"
 				(path "/1ee317a7-d9f9-4115-84b1-2928dd345c54/615c305d-8768-47e7-86f6-9adb9bcb9cb4"
-					(reference "#PWR066")
+					(reference "#PWR061")
 					(unit 1)
 				)
@@
 		(dnp no)
 		(fields_autoplaced yes)
-		(property "Reference" "#PWR060"
+		(property "Reference" "#PWR059"
 			(at 41.91 86.36 0)
 			(effects
@@
 			(project "Beyond_CMoy"
 				(path "/1ee317a7-d9f9-4115-84b1-2928dd345c54/615c305d-8768-47e7-86f6-9adb9bcb9cb4"
-					(reference "#PWR060")
+					(reference "#PWR059")
 					(unit 1)
 				)
@@
 		(on_board yes)
 		(dnp no)
-		(property "Reference" "U8"
+		(property "Reference" "U7"
 			(at 234.95 129.54 0)
 			(effects
@@
 			(project ""
 				(path "/1ee317a7-d9f9-4115-84b1-2928dd345c54/615c305d-8768-47e7-86f6-9adb9bcb9cb4"
-					(reference "U8")
+					(reference "U7")
 					(unit 1)
 				)
@@
 			)
 		)
-		(property "Footprint" "Diode_SMD:D_SOD-923"
+		(property "Footprint" "0_Devices:D_SOD-923_Edited"
 			(at 73.025 60.96 0)
 			(effects
@@
 		(dnp no)
 		(fields_autoplaced yes)
-		(property "Reference" "#PWR057"
+		(property "Reference" "#PWR056"
 			(at 190.5 74.93 0)
 			(effects
@@
 			(project "Beyond_CMoy"
 				(path "/1ee317a7-d9f9-4115-84b1-2928dd345c54/615c305d-8768-47e7-86f6-9adb9bcb9cb4"
-					(reference "#PWR057")
+					(reference "#PWR056")
 					(unit 1)
 				)
@@
 		(dnp no)
 		(fields_autoplaced yes)
-		(property "Reference" "#PWR053"
+		(property "Reference" "#PWR052"
 			(at 101.6 45.72 0)
 			(effects
@@
 			(project ""
 				(path "/1ee317a7-d9f9-4115-84b1-2928dd345c54/615c305d-8768-47e7-86f6-9adb9bcb9cb4"
-					(reference "#PWR053")
+					(reference "#PWR052")
 					(unit 1)
 				)
@@
 		(dnp no)
 		(fields_autoplaced yes)
-		(property "Reference" "R43"
+		(property "Reference" "R36"
 			(at 213.36 125.73 0)
 			(effects
@@
 			(project "Beyond_CMoy"
 				(path "/1ee317a7-d9f9-4115-84b1-2928dd345c54/615c305d-8768-47e7-86f6-9adb9bcb9cb4"
-					(reference "R43")
+					(reference "R36")
 					(unit 1)
 				)
@@
 		(dnp no)
 		(fields_autoplaced yes)
-		(property "Reference" "R39"
+		(property "Reference" "R32"
 			(at 71.12 68.58 0)
 			(effects
@@
 			(project "Beyond_CMoy"
 				(path "/1ee317a7-d9f9-4115-84b1-2928dd345c54/615c305d-8768-47e7-86f6-9adb9bcb9cb4"
-					(reference "R39")
+					(reference "R32")
 					(unit 1)
 				)
@@
 		(dnp no)
 		(fields_autoplaced yes)
-		(property "Reference" "R36"
+		(property "Reference" "R29"
 			(at 115.57 57.15 0)
 			(effects
@@
 			(project "Beyond_CMoy"
 				(path "/1ee317a7-d9f9-4115-84b1-2928dd345c54/615c305d-8768-47e7-86f6-9adb9bcb9cb4"
-					(reference "R36")
+					(reference "R29")
 					(unit 1)
 				)
@@
 		(dnp no)
 		(fields_autoplaced yes)
-		(property "Reference" "R38"
+		(property "Reference" "R31"
 			(at 62.23 68.58 0)
 			(effects
@@
 			(project "Beyond_CMoy"
 				(path "/1ee317a7-d9f9-4115-84b1-2928dd345c54/615c305d-8768-47e7-86f6-9adb9bcb9cb4"
-					(reference "R38")
+					(reference "R31")
 					(unit 1)
 				)
@@
 		(dnp no)
 		(fields_autoplaced yes)
-		(property "Reference" "#PWR054"
+		(property "Reference" "#PWR053"
 			(at 190.5 45.72 0)
 			(effects
@@
 			(project ""
 				(path "/1ee317a7-d9f9-4115-84b1-2928dd345c54/615c305d-8768-47e7-86f6-9adb9bcb9cb4"
-					(reference "#PWR054")
+					(reference "#PWR053")
 					(unit 1)
 				)
@@
 		(dnp no)
 		(fields_autoplaced yes)
-		(property "Reference" "R44"
+		(property "Reference" "R37"
 			(at 186.69 142.24 0)
 			(effects
@@
 			(project "Beyond_CMoy"
 				(path "/1ee317a7-d9f9-4115-84b1-2928dd345c54/615c305d-8768-47e7-86f6-9adb9bcb9cb4"
-					(reference "R44")
+					(reference "R37")
 					(unit 1)
 				)
@@
 		(dnp no)
 		(fields_autoplaced yes)
-		(property "Reference" "#PWR061"
+		(property "Reference" "#PWR060"
 			(at 113.03 118.11 0)
 			(effects
@@
 			(project "Beyond_CMoy"
 				(path "/1ee317a7-d9f9-4115-84b1-2928dd345c54/615c305d-8768-47e7-86f6-9adb9bcb9cb4"
-					(reference "#PWR061")
+					(reference "#PWR060")
 					(unit 1)
 				)
@@
 		(dnp no)
 		(fields_autoplaced yes)
-		(property "Reference" "TP5"
+		(property "Reference" "TP7"
 			(at 83.82 39.878 0)
 			(effects
@@
 			(project "Beyond_CMoy"
 				(path "/1ee317a7-d9f9-4115-84b1-2928dd345c54/615c305d-8768-47e7-86f6-9adb9bcb9cb4"
-					(reference "TP5")
+					(reference "TP7")
 					(unit 1)
 				)
@@
 		(dnp no)
 		(fields_autoplaced yes)
-		(property "Reference" "R37"
+		(property "Reference" "R30"
 			(at 193.04 58.42 0)
 			(effects
@@
 			(project ""
 				(path "/1ee317a7-d9f9-4115-84b1-2928dd345c54/615c305d-8768-47e7-86f6-9adb9bcb9cb4"
-					(reference "R37")
+					(reference "R30")
 					(unit 1)
 				)
@@
 		(dnp no)
 		(fields_autoplaced yes)
-		(property "Reference" "R35"
+		(property "Reference" "R28"
 			(at 138.43 52.07 0)
 			(effects
@@
 			(project "Beyond_CMoy"
 				(path "/1ee317a7-d9f9-4115-84b1-2928dd345c54/615c305d-8768-47e7-86f6-9adb9bcb9cb4"
-					(reference "R35")
+					(reference "R28")
 					(unit 1)
 				)
@@
 		(dnp no)
 		(fields_autoplaced yes)
-		(property "Reference" "R40"
+		(property "Reference" "R33"
 			(at 115.57 92.71 0)
 			(effects
@@
 			(project "Beyond_CMoy"
 				(path "/1ee317a7-d9f9-4115-84b1-2928dd345c54/615c305d-8768-47e7-86f6-9adb9bcb9cb4"
-					(reference "R40")
+					(reference "R33")
 					(unit 1)
 				)
@@
 		(dnp no)
 		(fields_autoplaced yes)
-		(property "Reference" "#PWR064"
+		(property "Reference" "#PWR063"
 			(at 176.53 158.75 0)
 			(effects
@@
 			(project "Beyond_CMoy"
 				(path "/1ee317a7-d9f9-4115-84b1-2928dd345c54/615c305d-8768-47e7-86f6-9adb9bcb9cb4"
-					(reference "#PWR064")
+					(reference "#PWR063")
 					(unit 1)
 				)
@@
 		(dnp no)
 		(fields_autoplaced yes)
-		(property "Reference" "#PWR055"
+		(property "Reference" "#PWR054"
 			(at 135.89 74.93 0)
 			(effects
@@
 			(project "Beyond_CMoy"
 				(path "/1ee317a7-d9f9-4115-84b1-2928dd345c54/615c305d-8768-47e7-86f6-9adb9bcb9cb4"
-					(reference "#PWR055")
+					(reference "#PWR054")
 					(unit 1)
 				)
@@
 		(dnp no)
 		(fields_autoplaced yes)
-		(property "Reference" "R42"
+		(property "Reference" "R35"
 			(at 186.69 125.73 0)
 			(effects
@@
 			(project "Beyond_CMoy"
 				(path "/1ee317a7-d9f9-4115-84b1-2928dd345c54/615c305d-8768-47e7-86f6-9adb9bcb9cb4"
-					(reference "R42")
+					(reference "R35")
 					(unit 1)
 				)
@@
 		(dnp no)
 		(fields_autoplaced yes)
-		(property "Reference" "#PWR056"
+		(property "Reference" "#PWR055"
 			(at 179.07 74.93 0)
 			(effects
@@
 			(project "Beyond_CMoy"
 				(path "/1ee317a7-d9f9-4115-84b1-2928dd345c54/615c305d-8768-47e7-86f6-9adb9bcb9cb4"
-					(reference "#PWR056")
+					(reference "#PWR055")
 					(unit 1)
 				)
@@
 		(dnp no)
 		(fields_autoplaced yes)
-		(property "Reference" "U7"
+		(property "Reference" "U6"
 			(at 166.37 40.64 0)
 			(effects
@@
 			(project ""
 				(path "/1ee317a7-d9f9-4115-84b1-2928dd345c54/615c305d-8768-47e7-86f6-9adb9bcb9cb4"
-					(reference "U7")
+					(reference "U6")
 					(unit 1)
 				)
@@
 		(dnp no)
 		(fields_autoplaced yes)
-		(property "Reference" "R41"
+		(property "Reference" "R34"
 			(at 237.49 113.03 90)
 			(effects
@@
 			(project "Beyond_CMoy"
 				(path "/1ee317a7-d9f9-4115-84b1-2928dd345c54/615c305d-8768-47e7-86f6-9adb9bcb9cb4"
-					(reference "R41")
+					(reference "R34")
 					(unit 1)
 				)
@@
 		(dnp no)
 		(fields_autoplaced yes)
-		(property "Reference" "U9"
+		(property "Reference" "U8"
 			(at 213.36 144.78 90)
 			(effects
@@
 			(project ""
 				(path "/1ee317a7-d9f9-4115-84b1-2928dd345c54/615c305d-8768-47e7-86f6-9adb9bcb9cb4"
-					(reference "U9")
+					(reference "U8")
 					(unit 1)
 				)
@@
 		(dnp no)
 		(fields_autoplaced yes)
-		(property "Reference" "#PWR059"
+		(property "Reference" "#PWR057"
 			(at 231.14 74.93 0)
 			(effects
@@
 			(project "Beyond_CMoy"
 				(path "/1ee317a7-d9f9-4115-84b1-2928dd345c54/615c305d-8768-47e7-86f6-9adb9bcb9cb4"
-					(reference "#PWR059")
+					(reference "#PWR057")
 					(unit 1)
 				)
