File: Beyond_CMoy/Beyond_CMoy.kicad_sch (KiCad schematic)
At the start: 0 parts

Commit message: RELEASED
Other:
- sheet Interface ports: added L_COUP, R_COUP; removed L_INPUT, R_INPUT
Changed lines of the file:
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@@
-			)
-		)
-		(pin "L_INPUT" output
-			(at 107.95 99.06 0)
-			(effects
-				(font
-					(size 1.27 1.27)
-				)
-				(justify right)
-			)
-		)
-		(pin "R_INPUT" output
-			(at 107.95 104.14 0)
-			(effects
-				(font
-					(size 1.27 1.27)
-				)
-				(justify right)
 			)
 		)
@@
 			(effects
 				(font
+					(size 1.27 1.27)
+				)
+				(justify right)
+			)
+		)
+		(pin "L_COUP" output
+			(at 107.95 99.06 0)
+			(effects
+				(font
+					(size 1.27 1.27)
+				)
+				(justify right)
+			)
+		)
+		(pin "R_COUP" output
+			(at 107.95 104.14 0)
+			(effects
+				(font

Commit message: Update Doc and Same verison Release
Release v1.0 , Update Doc Files
Other:
- added sheet Revision History (RevisionHistory.kicad_sch)
