File: Beyond_CMoy/Power Management.kicad_sch (KiCad schematic)
At the start: 23 parts, among them Q1 MMBT3906, U5 AP3012, U6 BD50FA1FP3

Commit message: RELEASED
Parts:
- added TP6, TP8: GND, TestPoint:TestPoint_THTPad_1.5x1.5mm_Drill0.7mm, symbol Connector:TestPoint
- C29, C30, C31, C32, C33, C34: footprint 0_Devices:0_C_0805_PasteCustom -> 0_Devices:0_C_0805_Edited; Manufacturer Samsung -> SAMSUNG
- D6: footprint LED_SMD:LED_0603_1608Metric -> LED_SMD:LED_Kingbright_APA1606_1.6x0.6mm_Horizontal; Mf. Part Number LTST-C191TGKT -> LTST-S270KGKT
- L1: value 4.7uH -> 10u; footprint Inductor_SMD:L_0603_1608Metric -> 0_Devices:0_L_1008_Edited; Mf. Part Number LQM18PN4R7MFRL -> DFE252010F-100M=P2
Connections:
- net GND: now also TP6.1, TP8.1
Other:
- note added: "Side View"

Commit message: Debugging & New Rev.
Connections:
- net +5V: now also U6.1 (VO); no longer U6.3 (VO)
- net +9V: now also U6.3 (VCC); no longer U6.1 (VCC)
Other:
- note added: "USE FET"
- moved on the sheet: C32, TP1
Changed lines of the file:
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@@
 	(title_block
 		(title "Power Management System")
-		(rev "1.0")
+		(rev "1.1")
 		(company "Natchpai")
 	)
 	(rectangle
-		(start 57.15 38.1)
+		(start 46.99 38.1)
 		(end 248.92 106.68)
 		(stroke
@@
 		)
 	)
+	(circle
+		(center 92.71 73.66)
+		(radius 32.3788)
+		(stroke
+			(width 0)
+			(type default)
+			(color 255 0 0 1)
+		)
+		(fill
+			(type color)
+			(color 255 0 0 0.3)
+		)
+	)
 	(text "Boost Converter"
 		(exclude_from_sim no)
-		(at 72.39 102.87 0)
+		(at 67.31 102.87 0)
 		(effects
 			(font
@@
 		)
 	)
+	(text "USE FET"
+		(exclude_from_sim no)
+		(at 96.52 119.38 0)
+		(effects
+			(font
+				(size 12.7 12.7)
+				(thickness 0.762)
+				(bold yes)
+				(color 255 0 0 1)
+			)
+		)
+	)
 	(text "Side View"
 		(exclude_from_sim no)
@@
 	)
 	(junction
-		(at 83.82 54.61)
+		(at 69.85 54.61)
 		(diameter 0)
 		(color 0 0 0 0)
@@
 	)
 	(junction
-		(at 88.9 54.61)
+		(at 74.93 54.61)
 		(diameter 0)
 		(color 0 0 0 0)
@@
 	)
 	(junction
-		(at 78.74 54.61)
+		(at 64.77 54.61)
 		(diameter 0)
 		(color 0 0 0 0)
@@
 	(wire
 		(pts
-			(xy 78.74 54.61) (xy 83.82 54.61)
+			(xy 64.77 54.61) (xy 69.85 54.61)
 		)
 		(stroke
@@
 	(wire
 		(pts
-			(xy 88.9 52.07) (xy 88.9 54.61)
+			(xy 74.93 52.07) (xy 74.93 54.61)
 		)
 		(stroke
@@
 	(wire
 		(pts
-			(xy 83.82 54.61) (xy 88.9 54.61)
+			(xy 69.85 54.61) (xy 74.93 54.61)
 		)
 		(stroke
@@
 	(wire
 		(pts
-			(xy 73.66 54.61) (xy 78.74 54.61)
+			(xy 59.69 54.61) (xy 64.77 54.61)
 		)
 		(stroke
@@
 	(wire
 		(pts
-			(xy 83.82 54.61) (xy 83.82 62.23)
+			(xy 69.85 54.61) (xy 69.85 62.23)
 		)
 		(stroke
@@
 	(wire
 		(pts
-			(xy 83.82 69.85) (xy 83.82 73.66)
+			(xy 69.85 69.85) (xy 69.85 73.66)
 		)
 		(stroke
@@
 	(wire
 		(pts
-			(xy 88.9 54.61) (xy 96.52 54.61)
+			(xy 74.93 54.61) (xy 96.52 54.61)
 		)
 		(stroke
@@
 	(wire
 		(pts
-			(xy 78.74 49.53) (xy 78.74 54.61)
+			(xy 64.77 49.53) (xy 64.77 54.61)
 		)
 		(stroke
@@
 	(hierarchical_label "+BATT"
 		(shape input)
-		(at 73.66 54.61 180)
+		(at 59.69 54.61 180)
 		(effects
 			(font
@@
 	(symbol
 		(lib_id "Device:C")
-		(at 83.82 66.04 0)
+		(at 69.85 66.04 0)
 		(unit 1)
 		(exclude_from_sim no)
@@
 		(fields_autoplaced yes)
 		(property "Reference" "C32"
-			(at 87.63 64.77 0)
+			(at 73.66 64.77 0)
 			(effects
 				(font
@@
 		)
 		(property "Value" "1u"
-			(at 87.63 67.31 0)
+			(at 73.66 67.31 0)
 			(effects
 				(font
@@
 		)
 		(property "Footprint" "0_Devices:0_C_0805_Edited"
-			(at 84.7852 69.85 0)
+			(at 70.8152 69.85 0)
 			(effects
 				(font
@@
 		)
 		(property "Datasheet" "~"
-			(at 83.82 66.04 0)
+			(at 69.85 66.04 0)
 			(effects
 				(font
@@
 		)
 		(property "Description" "1μF/50Vdc, ±10%, X7R"
-			(at 83.82 66.04 0)
+			(at 69.85 66.04 0)
 			(effects
 				(font
@@
 		)
 		(property "Manufacturer" "SAMSUNG"
-			(at 83.82 66.04 0)
+			(at 69.85 66.04 0)
 			(effects
 				(font
@@
 		)
 		(property "Mf. Part Number" "CL21B105KBFNNNE"
-			(at 83.82 66.04 0)
+			(at 69.85 66.04 0)
 			(effects
 				(font
@@
 		(on_board yes)
 		(dnp no)
-		(fields_autoplaced yes)
 		(property "Reference" "Q1"
 			(at 101.6 67.31 90)
@@
 	(symbol
 		(lib_id "power:GND")
-		(at 83.82 73.66 0)
+		(at 69.85 73.66 0)
 		(unit 1)
 		(exclude_from_sim no)
@@
 		(fields_autoplaced yes)
 		(property "Reference" "#PWR047"
-			(at 83.82 80.01 0)
+			(at 69.85 80.01 0)
 			(effects
 				(font
@@
 		)
 		(property "Value" "GND"
-			(at 83.82 78.74 0)
+			(at 69.85 78.74 0)
 			(effects
 				(font
@@
 		)
 		(property "Footprint" ""
-			(at 83.82 73.66 0)
+			(at 69.85 73.66 0)
 			(effects
 				(font
@@
 		)
 		(property "Datasheet" ""
-			(at 83.82 73.66 0)
+			(at 69.85 73.66 0)
 			(effects
 				(font
@@
 		)
 		(property "Description" "Power symbol creates a global label with name \"GND\" , ground"
-			(at 83.82 73.66 0)
+			(at 69.85 73.66 0)
 			(effects
 				(font
@@
 	(symbol
 		(lib_id "Connector:TestPoint")
-		(at 88.9 52.07 0)
+		(at 74.93 52.07 0)
 		(unit 1)
 		(exclude_from_sim no)
@@
 		(fields_autoplaced yes)
 		(property "Reference" "TP1"
-			(at 91.44 47.498 0)
+			(at 77.47 47.498 0)
 			(effects
 				(font
@@
 		)
 		(property "Value" "+BATT"
-			(at 91.44 50.038 0)
+			(at 77.47 50.038 0)
 			(effects
 				(font
@@
 		)
 		(property "Footprint" "TestPoint:TestPoint_Pad_D2.0mm"
-			(at 93.98 52.07 0)
+			(at 80.01 52.07 0)
 			(effects
 				(font
@@
 		)
 		(property "Datasheet" "~"
-			(at 93.98 52.07 0)
+			(at 80.01 52.07 0)
 			(effects
 				(font
@@
 		)
 		(property "Description" "test point"
-			(at 88.9 52.07 0)
+			(at 74.93 52.07 0)
 			(effects
 				(font
@@
 		)
 		(property "Manufacturer" ""
-			(at 88.9 52.07 0)
+			(at 74.93 52.07 0)
 			(effects
 				(font
@@
 		)
 		(property "Mf. Part Number" ""
-			(at 88.9 52.07 0)
+			(at 74.93 52.07 0)
 			(effects
 				(font
@@
 	(symbol
 		(lib_id "power:+BATT")
-		(at 78.74 49.53 0)
+		(at 64.77 49.53 0)
 		(unit 1)
 		(exclude_from_sim no)
@@
 		(fields_autoplaced yes)
 		(property "Reference" "#PWR041"
-			(at 78.74 53.34 0)
+			(at 64.77 53.34 0)
 			(effects
 				(font
@@
 		)
 		(property "Value" "+BATT"
-			(at 78.74 44.45 0)
+			(at 64.77 44.45 0)
 			(effects
 				(font
@@
 		)
 		(property "Footprint" ""
-			(at 78.74 49.53 0)
+			(at 64.77 49.53 0)
 			(effects
 				(font
@@
 		)
 		(property "Datasheet" ""
-			(at 78.74 49.53 0)
+			(at 64.77 49.53 0)
 			(effects
 				(font
@@
 		)
 		(property "Description" "Power symbol creates a global label with name \"+BATT\""
-			(at 78.74 49.53 0)
+			(at 64.77 49.53 0)
 			(effects
 				(font

Commit message: Re-layout
Parts:
- removed Q1: MMBT3906, Package_TO_SOT_SMD:SOT-23, symbol Transistor_BJT:MMBT3906
- removed R31: 10k, Resistor_SMD:R_0603_1608Metric, symbol Device:R
- removed U6: BD50FA1FP3, Package_TO_SOT_SMD:SOT-89-3, symbol Regulator_Linear:BD50FC0FP
- added C31: 0.1u, Capacitor_SMD:C_0402_1005Metric, symbol Device:C
- added Q1: AO3401A, Package_TO_SOT_SMD:SOT-23-3, symbol Transistor_FET:AO3401A
- added U5: BD50FA1FP3-ZTL, Package_TO_SOT_SMD:SOT-89-3, symbol BD50FA1FP3-ZTL:BD50FA1FP3-ZTL
- R23: renamed from R29; value 0 -> 1M; now fitted
- R27: renamed from R34; value 5.1k -> 0
- TP5: renamed from TP4; footprint TestPoint:TestPoint_Pad_D2.0mm -> TestPoint:TestPoint_Pad_D1.0mm
- renumbered C30 to C28, C31 to C29, C29 to C30, R30 to R24, R33 to R25, R32 to R26, TP2 to TP1, TP1 to TP2, TP6 to TP3, TP3 to TP4, TP8 to TP6, U5 to U4
Connections:
- net +5V: now also U5.1 (VO)
- net +9V: now also U5.3 (VCC)
- net +BATT: now also R23.1, C31.1, Q1.2 (S); no longer C32.1, L1.1, R23.2, U4.5 (IN)
- net GND: now also U5.2 (GND)
- net FET_G: now reaches R27.1
- net FET_G: now also R23.2, C31.2, Q1.1 (G)
- net BS_EN renamed ON_BATT
- net ON_BATT: now also C32.1, L1.1, U4.5 (IN), Q1.3 (D); no longer R23.1
Other:
- note removed: "USE FET"
- moved on the sheet: C30, C32, R25, R26, R27, TP2, TP3
