File: Beyond_CMoy/RevisionHistory.kicad_sch (KiCad schematic)
At the start: 0 parts

Commit message: Debugging & New Rev.
Other:
- note added: "1.1"
- note added: "19/Nov/2025"
- note added: "Changed U6's Symbol and Pin Number"
- note added: "First version Schematic/PCB Release"
- note removed: "0.1"
- note removed: "22/Nov/2025"
- note removed: "Author"
- note removed: "Date"
- note removed: "Description"
- note removed: "First version SCH/PCB Release"
- note removed: "Initial project"
- note removed: "Natchanon T."

Commit message: Re-layout
Other:
- note added: "21/Nov/2025"
- note added: "Interface * Added 33pF on (R_BT) and (L_BT) Line Amplifier * Redesign Buffer stage * Changed DC Gain=2 Power Management System * Use MOSFET as a switch to power up the module. * Changed BD50FA1FP3(5V Regulator) Pin Alignment Battery Management System * Increased ESD9L5.0ST5G Footprint size - Changed Alignment of Ref. Designators"
- note removed: "19/Nov/2025"
- note removed: "Changed U6's Symbol and Pin Number"
Changed lines of the file:
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@@
 	(text "First version Schematic/PCB Release"
 		(exclude_from_sim no)
-		(at 33.02 43.18 0)
-		(effects
-			(font
-				(size 2.032 2.032)
+		(at 29.21 39.37 0)
+		(effects
+			(font
+				(face "Calibri")
+				(size 1.778 1.778)
 				(color 0 0 0 1)
 			)
@@
 		)
 	)
-	(text "Changed U6's Symbol and Pin Number"
-		(exclude_from_sim no)
-		(at 33.02 62.23 0)
-		(effects
-			(font
-				(size 2.032 2.032)
+	(text "Interface\n* Added 33pF on (R_BT) and (L_BT) Line\n\nAmplifier\n* Redesign Buffer stage\n* Changed DC Gain=2\n\nPower Management System\n* Use MOSFET as a switch to power up the module.\n* Changed BD50FA1FP3(5V Regulator) Pin Alignment\n\nBattery Management System\n* Increased ESD9L5.0ST5G Footprint size\n\n- Changed Alignment of Ref. Designators"
+		(exclude_from_sim no)
+		(at 29.21 55.88 0)
+		(effects
+			(font
+				(face "Calibri")
+				(size 1.778 1.778)
+				(color 0 0 0 1)
+			)
+			(justify left top)
+		)
+	)
+	(text "21/Nov/2025"
+		(exclude_from_sim no)
+		(at 83.82 50.8 0)
+		(effects
+			(font
+				(size 2.032 2.032)
+				(thickness 0.4064)
+				(bold yes)
 				(color 0 0 0 1)
 			)
@@
 		)
 	)
-	(text "19/Nov/2025"
-		(exclude_from_sim no)
-		(at 87.63 54.61 0)
+	(text "07/Dec/2025"
+		(exclude_from_sim no)
+		(at 83.82 33.02 0)
 		(effects
 			(font
@@
 		)
 	)
-	(text "07/Dec/2025"
-		(exclude_from_sim no)
-		(at 87.63 36.83 0)
-		(effects
-			(font
-				(size 2.032 2.032)
-				(thickness 0.4064)
-				(bold yes)
-				(color 0 0 0 1)
-			)
-			(justify left)
-		)
-	)
 	(text "1.0"
 		(exclude_from_sim no)
-		(at 45.72 36.83 0)
+		(at 41.91 33.02 0)
 		(effects
 			(font
@@
 	(text "Revision"
 		(exclude_from_sim no)
-		(at 36.83 36.83 0)
+		(at 33.02 33.02 0)
 		(effects
 			(font
@@
 	(text "Revision"
 		(exclude_from_sim no)
-		(at 36.83 54.61 0)
+		(at 33.02 50.8 0)
 		(effects
 			(font
@@
 		)
 	)
-	(text "1.1"
-		(exclude_from_sim no)
-		(at 45.72 54.61 0)
-		(effects
-			(font
-				(size 2.032 2.032)
-				(thickness 0.4064)
-				(bold yes)
-				(color 0 0 0 1)
-			)
-		)
-	)
-	(polyline
-		(pts
-			(xy 29.21 57.15) (xy 105.41 57.15)
-		)
-		(stroke
-			(width 0.254)
-			(type default)
-			(color 0 0 0 1)
-		)
-	)
-	(polyline
-		(pts
-			(xy 29.21 50.8) (xy 105.41 50.8)
-		)
-		(stroke
-			(width 0.254)
-			(type default)
-			(color 0 0 0 1)
-		)
-	)
-	(polyline
-		(pts
-			(xy 29.21 33.02) (xy 29.21 165.1)
-		)
-		(stroke
-			(width 0.254)
-			(type default)
-			(color 0 0 0 1)
-		)
-	)
-	(polyline
-		(pts
-			(xy 29.21 33.02) (xy 105.41 33.02)
-		)
-		(stroke
-			(width 0.254)
-			(type default)
-			(color 0 0 0 1)
-		)
-	)
-	(polyline
-		(pts
-			(xy 29.21 39.37) (xy 105.41 39.37)
-		)
-		(stroke
+	(text "1.1\n"
+		(exclude_from_sim no)
+		(at 41.91 50.8 0)
+		(effects
+			(font
+				(size 2.032 2.032)
+				(thickness 0.4064)
+				(bold yes)
+				(color 0 0 0 1)
+			)
+		)
+	)
+	(polyline
+		(pts
+			(xy 110.49 29.21) (xy 110.49 161.29)
+		)
+		(stroke
+			(width 0.254)
+			(type default)
+			(color 0 0 0 1)
+		)
+	)
+	(polyline
+		(pts
+			(xy 271.78 29.21) (xy 271.78 161.29)
+		)
+		(stroke
+			(width 0.254)
+			(type default)
+			(color 0 0 0 1)
+		)
+	)
+	(polyline
+		(pts
+			(xy 101.6 29.21) (xy 101.6 161.29)
+		)
+		(stroke
+			(width 0.254)
+			(type default)
+			(color 0 0 0 1)
+		)
+	)
+	(polyline
+		(pts
+			(xy 25.4 53.34) (xy 101.6 53.34)
+		)
+		(stroke
+			(width 0.254)
+			(type default)
+			(color 0 0 0 1)
+		)
+	)
+	(polyline
+		(pts
+			(xy 195.58 29.21) (xy 271.78 29.21)
+		)
+		(stroke
+			(width 0.254)
+			(type default)
+			(color 0 0 0 1)
+		)
+	)
+	(polyline
+		(pts
+			(xy 25.4 161.29) (xy 101.6 161.29)
+		)
+		(stroke
+			(width 0.254)
+			(type default)
+			(color 0 0 0 1)
+		)
+	)
+	(polyline
+		(pts
+			(xy 25.4 46.99) (xy 101.6 46.99)
+		)
+		(stroke
+			(width 0.254)
+			(type default)
+			(color 0 0 0 1)
+		)
+	)
+	(polyline
+		(pts
+			(xy 110.49 29.21) (xy 186.69 29.21)
+		)
+		(stroke
+			(width 0.254)
+			(type default)
+			(color 0 0 0 1)
+		)
+	)
+	(polyline
+		(pts
+			(xy 186.69 29.21) (xy 186.69 161.29)
+		)
+		(stroke
+			(width 0.254)
+			(type default)
+			(color 0 0 0 1)
+		)
+	)
+	(polyline
+		(pts
+			(xy 110.49 161.29) (xy 186.69 161.29)
+		)
+		(stroke
+			(width 0.254)
+			(type default)
+			(color 0 0 0 1)
+		)
+	)
+	(polyline
+		(pts
+			(xy 195.58 29.21) (xy 195.58 161.29)
+		)
+		(stroke
+			(width 0.254)
+			(type default)
+			(color 0 0 0 1)
+		)
+	)
+	(polyline
+		(pts
+			(xy 25.4 29.21) (xy 25.4 161.29)
+		)
+		(stroke
+			(width 0.254)
+			(type default)
+			(color 0 0 0 1)
+		)
+	)
+	(polyline
+		(pts
+			(xy 25.4 29.21) (xy 101.6 29.21)
+		)
+		(stroke
+			(width 0.254)
+			(type default)
+			(color 0 0 0 1)
+		)
+	)
+	(polyline
+		(pts
+			(xy 195.58 161.29) (xy 271.78 161.29)
+		)
+		(stroke
+			(width 0.254)
+			(type default)
+			(color 0 0 0 1)
+		)
+	)
+	(polyline
+		(pts
+			(xy 25.4 35.56) (xy 101.6 35.56)
+		)
+		(stroke
