File: Beyond_CMoy/interface.kicad_sch (KiCad schematic)
At the start: 18 parts, among them J1 PJ-327F, J2 Conn_01x04_Socket, J3 PJ-327F, P1 10k

Commit message: RELEASED
Parts:
- J2: Manufacturer (none) -> -
Connections:
- net GND: now also P1.8; no longer P1.7
- net Power_ON: now also P1.7; no longer P1.8
- net L_INPUT renamed L_COUP
- net R_INPUT renamed R_COUP
Other:
- moved on the sheet: P1C
Changed lines of the file:
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@@
 		(stroke
 			(width 0.508)
-			(type default)
+			(type solid)
 			(color 194 194 194 1)
 		)
 		(fill
-			(type color)
-			(color 255 255 255 1)
+			(type none)
 		)
 	)
@@
 		(stroke
 			(width 0.508)
-			(type default)
+			(type solid)
 			(color 194 194 194 1)
 		)
 		(fill
-			(type color)
-			(color 255 255 255 1)
+			(type none)
 		)
 	)
@@
 		(stroke
 			(width 0.508)
-			(type default)
+			(type solid)
 			(color 194 194 194 1)
 		)
 		(fill
-			(type color)
-			(color 255 255 255 1)
+			(type none)
 		)
 	)
@@
 		(stroke
 			(width 0.508)
-			(type default)
+			(type solid)
 			(color 194 194 194 1)
 		)
 		(fill
-			(type color)
-			(color 255 255 255 1)
+			(type none)
 		)
 	)
@@
 		)
 	)
-	(hierarchical_label "R_INPUT"
+	(hierarchical_label "R_COUP"
 		(shape output)
 		(at 210.82 66.04 0)
@@
 		)
 	)
-	(hierarchical_label "L_INPUT"
+	(hierarchical_label "L_COUP"
 		(shape output)
 		(at 210.82 57.15 0)
@@
 			)
 		)
+		(property "Manufacturer" "-"
+			(at 78.74 58.42 0)
+			(effects
+				(font
+					(size 1.27 1.27)
+				)
+				(hide yes)
+			)
+		)
 		(pin "3"
 		)
@@
 	(symbol
 		(lib_id "0_Potentiometer:RK097GS")
-		(at 43.18 171.45 0)
+		(at 43.18 171.45 180)
 		(unit 3)
 		(exclude_from_sim no)
@@
 		(fields_autoplaced yes)
 		(property "Reference" "P1"
-			(at 44.45 171.45 0)
+			(at 45.72 171.45 0)
 			(effects
 				(font
@@
 					(thickness 0.1588)
 				)
-				(justify left)
+				(justify right)
 			)
 		)
 		(property "Value" "10k"
-			(at 44.45 172.72 0)
+			(at 41.91 170.18 0)
 			(effects
 				(font
@@
 		)
 		(property "Footprint" "0_Potentiometer:0_RK097GS_Dual_Horizontal_Switch"
-			(at 44.45 181.864 0)
+			(at 41.91 161.036 0)
 			(effects
 				(font

Commit message: Update Doc and Same verison Release
Release v1.0 , Update Doc Files
Parts:
- J2: Mf. Part Number (none) -> -

Commit message: Re-layout
Parts:
- added C2, C4: 33p, Capacitor_SMD:C_0402_1005Metric, symbol Device:C
- renumbered C2 to C3, C3 to C5, C4 to C6, C5 to C7, C6 to C8, J2 to J1, J1 to J2
Connections:
- net GND: now also C2.2, C4.2
- net L_BT: now also C2.1
- net R_BT: now also C4.1
Other:
- moved on the sheet: C1, C3, C5, C6, C7, C8, D1, D2, D3, D4, J1, J2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
